File: mainboard/invaderBoard.sch (KiCad schematic (older format))
At the start: 4 parts

Commit message: Notes to PCB design
Parts:
- P?: symbol invaderBoard-rescue:CONN_01X02 -> invaderBoard-rescue:CONN_01X02-invaderBoard-rescue
- P?: symbol invaderBoard-rescue:CONN_01X03 -> invaderBoard-rescue:CONN_01X03-invaderBoard-rescue
- Q? (x2): symbol invaderBoard-rescue:IRF540N -> invaderBoard-rescue:IRF540N-invaderBoard-rescue
Other:
- note added: "FUSE!\nLipo Master Disable (latching, so it is off by default but turns on during power-up)\nOn-off button\n\nConn for motor drivers, lipo, lipo balance output, aux. outputs\nArduino vs. esp32?\n"
Changed lines of the file:
@@
 $EndDescr
 $Comp
-L invaderBoard-rescue:CONN_01X02 P?
+L invaderBoard-rescue:CONN_01X02-invaderBoard-rescue P?
 U 1 1 5CC6A607
 P 2300 2125
@@
 $EndComp
 $Comp
-L invaderBoard-rescue:CONN_01X03 P?
+L invaderBoard-rescue:CONN_01X03-invaderBoard-rescue P?
 U 1 1 5CC6A69C
 P 2275 2875
@@
 $EndComp
 $Comp
-L invaderBoard-rescue:IRF540N Q?
+L invaderBoard-rescue:IRF540N-invaderBoard-rescue Q?
 U 1 1 5CC6A70B
 P 4700 2200
@@
 $EndComp
 $Comp
-L invaderBoard-rescue:IRF540N Q?
+L invaderBoard-rescue:IRF540N-invaderBoard-rescue Q?
 U 1 1 5CC6A75C
 P 5900 2200
@@
 	1    0    0    -1
 $EndComp
+Text Notes 4200 4100 0    50   ~ 0
+FUSE!\nLipo Master Disable (latching, so it is off by default but turns on during power-up)\nOn-off button\n\nConn for motor drivers, lipo, lipo balance output, aux. outputs\nArduino vs. esp32?\n
 $EndSCHEMATC
