File: mainboard/invaderBoard.kicad_pcb (KiCad board)
At the start: 2 copper layers, 50 x 100 mm, 30 parts, among them J1 Conn_01x02, J10 Conn_01x03, J11 Conn_01x04, J13 Conn_01x03, J19 Conn_01x02, J2 USB_A, J20 Conn_01x02, J3 Conn_01x04, J4 Conn_02x04_Odd_Even, J5 Conn_02x04_Odd_Even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

Commit message: arduino FW added + some changes on sch.
Parts:
- J1: footprint Connector_Wire:SolderWirePad_1x02_P7.62mm_Drill2mm -> .pretty:BiggerSolderPad
- moved J1 2.09 mm to (212.0, 67.0)
Routing:
- net Net-(F1-Pad2): track 15.0 -> 11.1 mm
- net /HV: track 197.9 -> 197.0 mm
Changed lines of the file:
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@@
     (thickness 1.6)
     (drawings 12)
-    (tracks 292)
+    (tracks 293)
     (zones 0)
     (modules 30)
@@
   )
   (setup
-    (last_trace_width 0.25)
+    (last_trace_width 1.524)
     (user_trace_width 0.508)
     (user_trace_width 1.016)
@@
     (add_net "Net-(F1-Pad2)")
   )
+  (module .pretty:BiggerSolderPad (layer F.Cu)
+    (at 212 67)
+    (descr "Wire solder connection")
+    (tags connector)
+    (attr virtual)
+    (fp_text reference J1 (at 3.81 -5.08) (layer F.SilkS)
+      (effects (font (size 1 1) (thickness 0.15)))
+    )
+    (fp_text value Conn_01x02 (at 3.81 4.445) (layer F.Fab)
+      (effects (font (size 1 1) (thickness 0.15)))
+    )
+    (fp_line (start 11.12 3.5) (end -3.5 3.5) (layer F.CrtYd) (width 0.05))
+    (fp_line (start 11.12 3.5) (end 11.12 -3.5) (layer F.CrtYd) (width 0.05))
+    (fp_line (start -3.5 -3.5) (end -3.5 3.5) (layer F.CrtYd) (width 0.05))
+    (fp_line (start -3.5 -3.5) (end 11.12 -3.5) (layer F.CrtYd) (width 0.05))
+    (fp_text user %R (at 3.81 0) (layer F.Fab)
+      (effects (font (size 1 1) (thickness 0.15)))
+    )
+    (pad 2 thru_hole circle (at 11 0) (size 8 8) (drill 4) (layers *.Cu *.Mask)
+      (net 1 "Net-(F1-Pad2)"))
+    (pad 1 thru_hole rect (at 0 0) (size 8 8) (drill 4) (layers *.Cu *.Mask)
+      (net 2 /HV))
+  )
   (module MountingHole:MountingHole_3.2mm_M3 (layer F.Cu)
     (at 250 50)
@@
     (pad 1 thru_hole circle (at 0 0 180) (size 2 2) (drill 1) (layers *.Cu *.Mask)
       (net 27 "Net-(F1-Pad1)"))
-  )
-  (module Connector_Wire:SolderWirePad_1x02_P7.62mm_Drill2mm (layer F.Cu)
-    (at 212.09 69.088)
-    (descr "Wire solder connection")
-    (tags connector)
-    (attr virtual)
-    (fp_text reference J1 (at 3.175 -3.81) (layer F.SilkS)
-      (effects (font (size 1 1) (thickness 0.15)))
-    )
-    (fp_text value Conn_01x02 (at 3.175 3.81) (layer F.Fab)
-      (effects (font (size 1 1) (thickness 0.15)))
-    )
-    (fp_line (start 9.09 2.75) (end -2.75 2.75) (layer F.CrtYd) (width 0.05))
-    (fp_line (start 9.09 2.75) (end 9.09 -2.75) (layer F.CrtYd) (width 0.05))
-    (fp_line (start -2.75 -2.75) (end -2.75 2.75) (layer F.CrtYd) (width 0.05))
-    (fp_line (start -2.75 -2.75) (end 9.09 -2.75) (layer F.CrtYd) (width 0.05))
-    (fp_text user %R (at 3.175 0) (layer F.Fab)
-      (effects (font (size 1 1) (thickness 0.15)))
-    )
-    (pad 2 thru_hole circle (at 6.35 0) (size 4.50088 4.50088) (drill 1.99898) (layers *.Cu *.Mask)
-      (net 1 "Net-(F1-Pad2)"))
-    (pad 1 thru_hole rect (at 0 0) (size 4.50088 4.50088) (drill 1.99898) (layers *.Cu *.Mask)
-      (net 2 /HV))
   )
   (module Resistor_SMD:R_0805_2012Metric_Pad1.15x1.40mm_HandSolder (layer B.Cu)
@@
   (gr_line (start 216.408 51.435) (end 216.408 48.895) (layer Edge.Cuts) (width 0.05))
   (gr_line (start 210.693 51.435) (end 216.408 51.435) (layer Edge.Cuts) (width 0.05))
-  (segment (start 225.298 62.23) (end 225.298 56.896) (width 1.524) (layer F.Cu) (net 1))
-  (segment (start 218.44 69.088) (end 225.298 62.23) (width 1.524) (layer F.Cu) (net 1))
+  (segment (start 223 67) (end 223 62.5) (width 1.524) (layer F.Cu) (net 1))
+  (segment (start 225.298 60.202) (end 225.298 59.702) (width 1.524) (layer F.Cu) (net 1))
+  (segment (start 223 62.5) (end 225.298 60.202) (width 1.524) (layer F.Cu) (net 1))
+  (segment (start 225.298 56.896) (end 225.298 59.702) (width 1.524) (layer F.Cu) (net 1))
   (segment (start 207.645 113.03) (end 208.534 113.03) (width 1.016) (layer F.Cu) (net 2))
   (segment (start 208.534 113.03) (end 210.185 113.03) (width 1.016) (layer F.Cu) (net 2))
@@
   (segment (start 234.442 40.64) (end 234.442 41.148) (width 1.524) (layer F.Cu) (net 2))
   (segment (start 234.442 41.148) (end 232.156 43.434) (width 1.524) (layer F.Cu) (net 2))
-  (segment (start 212.09 64.262) (end 212.09 69.088) (width 1.524) (layer B.Cu) (net 2))
   (segment (start 222.504 43.434) (end 219.71 46.228) (width 1.524) (layer B.Cu) (net 2))
   (segment (start 232.156 43.434) (end 222.504 43.434) (width 1.524) (layer B.Cu) (net 2))
-  (segment (start 219.71 46.228) (end 219.71 60.96) (width 1.524) (layer B.Cu) (net 2))
-  (segment (start 217.932 62.738) (end 213.614 62.738) (width 1.524) (layer B.Cu) (net 2))
-  (segment (start 219.71 60.96) (end 217.932 62.738) (width 1.524) (layer B.Cu) (net 2))
-  (segment (start 213.614 62.738) (end 212.09 64.262) (width 1.524) (layer B.Cu) (net 2))
-  (segment (start 230.34 65.024) (end 228.562 63.246) (width 1.016) (layer B.Cu) (net 2))
-  (segment (start 232.156 65.024) (end 230.34 65.024) (width 1.016) (layer B.Cu) (net 2))
-  (segment (start 221.996 63.246) (end 219.71 60.96) (width 1.016) (layer B.Cu) (net 2))
-  (segment (start 228.562 63.246) (end 221.996 63.246) (width 1.016) (layer B.Cu) (net 2))
   (segment (start 209.296 112.776) (end 209.042 113.03) (width 1.524) (layer F.Cu) (net 2))
   (segment (start 212.09 72.86244) (end 209.296 75.65644) (width 1.524) (layer F.Cu) (net 2))
@@
   (segment (start 226.748 111.252) (end 225.552 111.252) (width 1.016) (layer B.Cu) (net 2))
   (segment (start 227.076 118.872) (end 227.974 117.974) (width 1.016) (layer B.Cu) (net 2))
+  (segment (start 212 67) (end 212 64) (width 1.524) (layer B.Cu) (net 2))
+  (segment (start 212 64) (end 214.5 61.5) (width 1.524) (layer B.Cu) (net 2))
+  (segment (start 218.5 61.5) (end 219.71 60.29) (width 1.524) (layer B.Cu) (net 2))
+  (segment (start 214.5 61.5) (end 218.5 61.5) (width 1.524) (layer B.Cu) (net 2))
+  (segment (start 219.71 46.228) (end 219.71 60.29) (width 1.524) (layer B.Cu) (net 2))
+  (segment (start 232.156 63.208) (end 232.156 65.024) (width 1.016) (layer B.Cu) (net 2))
+  (segment (start 229.238 60.29) (end 232.156 63.208) (width 1.016) (layer B.Cu) (net 2))
+  (segment (start 219.71 60.29) (end 229.238 60.29) (width 1.016) (layer B.Cu) (net 2))
   (segment (start 213.48 88.265) (end 213.36 88.145) (width 1.016) (layer B.Cu) (net 3))
   (segment (start 218.939 88.265) (end 213.48 88.265) (width 1.016) (layer B.Cu) (net 3))

Commit message: PCB updated -v1 finalized
Connections:
- J2 pad 2: (no net) -> Net-(J2-Pad2)
- J2 pad 3: (no net) -> Net-(J2-Pad3)
- J3 pad 1: (no net) -> Net-(J3-Pad1)
- J4 pad 5: (no net) -> Net-(J4-Pad5)
- J4 pad 6: (no net) -> Net-(J4-Pad6)
- J5 pad 5: (no net) -> Net-(J5-Pad5)
- J5 pad 6: (no net) -> Net-(J5-Pad6)
- U3 pad 1: (no net) -> /M1_LPWM
- U3 pad 10: (no net) -> Net-(U3-Pad10)
- U3 pad 11: (no net) -> Net-(U3-Pad11)
- U3 pad 12: (no net) -> Net-(U3-Pad12)
- U3 pad 13: (no net) -> Net-(U3-Pad13)
- U3 pad 16: (no net) -> /USER_MISO
- U3 pad 17: (no net) -> /USER_SCK
- U3 pad 18: (no net) -> /USER_MOSI
- U3 pad 19: (no net) -> /USER_SS
- U3 pad 2: (no net) -> Net-(U3-Pad2)
- U3 pad 22: (no net) -> Net-(U3-Pad22)
- U3 pad 24: (no net) -> /USER_SDA
- U3 pad 25: (no net) -> /USER_SCL
- U3 pad 3: (no net) -> Net-(U3-Pad3)
- U3 pad 34: /M1_LPWM -> Net-(U3-Pad34)
Routing:
- net /M1_LPWM: track 13.1 -> 27.0 mm
